Commit message: docs(water): 修复ROV文档公式渲染与演示,响应评审意见
- 公式语法统一为 \(...\)/\[...\],配合可达CDN(bootcdn)修复公式不渲染
- 4.3键盘控制删除重复按键表,改跳转链接,聚焦目标跟踪
- 补充动图引用;动图压缩至4.34MB(<5MB)
- 新增本地 mermaid.min.js,系统架构图离线渲染
- 补充ROV模型惯性参数、相机传感器等代码优化

File: src/water/rov_gazebo_sim/urdf/simple_rov.urdf (robot description, URDF)
Before this commit: robot simple_rov, 2 links, 1 joints
Links:
- link base_link: mass None -> 10
- link camera_link: mass None -> 0.1
