Commit message: fix(humanoid): 修复人形机器人运动控制并重录正确演示动图
- 重录演示动图:机器人从起点走向红色目标(243KB,<5MB)

- 修正 spawn 位置避免机器人陷地,删除 world 重叠冗余模型

- URDF 添加左右轮与 diff_drive 插件,驱动 /humanoid/cmd_vel

- perception 修正摄像头话题名为 camera_sensor/image_raw

File: src/humanoid/humanoid_gazebo_sim/urdf/simple_humanoid.urdf (robot description, URDF)
Before this commit: robot simple_humanoid, 3 links, 2 joints
Links:
- added link left_wheel_link, mass 0.1; collision cylinder length=0.06 radius=0.1; visual cylinder length=0.06 radius=0.1
- added link right_wheel_link, mass 0.1; collision cylinder length=0.06 radius=0.1; visual cylinder length=0.06 radius=0.1
Joints:
- added joint left_wheel_joint: type continuous, parent base_link, child left_wheel_link, origin xyz=0 0.15 -0.25 rpy=1.5708 0 0, axis 1 0 0
- added joint right_wheel_joint: type continuous, parent base_link, child right_wheel_link, origin xyz=0 -0.15 -0.25 rpy=1.5708 0 0, axis 1 0 0
